File: Hardware/Cube_UCarrierBoard/PSM.kicad_sch (KiCad schematic)
At the start: 60 parts, among them Q1 Q_Dual_PMOS, Q2 Q_Dual_PMOS, Q3 Q_Dual_PMOS, Q4 MMBT3906-TPCT-ND, U1 BQ24315, U2 BQ24315, U3 LTC4417 QFN, U4 MIC5332, U5 LT3469ETS8PBF, U6 BQ24313

Commit message: Fixed some footprints
Parts:
- L1: footprint Fuse:Fuse_0603_1608Metric -> libraries:C_FEEDTHRU_0603_TDK
- Q1, Q2, Q3: footprint libraries:RESCAXE64P320X160X70-10N -> (none)
- U5: footprint Linear_Technology-LT3469ETS8PBF-* -> Package_TO_SOT_SMD:TSOT-23-8
Changed lines of the file:
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@@
     (property "Reference" "Q2" (id 0) (at 165.1 52.5485 90))
     (property "Value" "Q_Dual_PMOS" (id 1) (at 165.1 55.3236 90))
-    (property "Footprint" "libraries:RESCAXE64P320X160X70-10N" (id 2) (at 165.1 59.69 0)
+    (property "Footprint" "" (id 2) (at 165.1 59.69 0)
       (effects (font (size 1.27 1.27)) hide)
     )
@@
     (property "Reference" "Q1" (id 0) (at 139.7 34.7685 90))
     (property "Value" "Q_Dual_PMOS" (id 1) (at 139.7 37.5436 90))
-    (property "Footprint" "libraries:RESCAXE64P320X160X70-10N" (id 2) (at 139.7 41.91 0)
+    (property "Footprint" "" (id 2) (at 139.7 41.91 0)
       (effects (font (size 1.27 1.27)) hide)
     )
@@
     (property "Reference" "U5" (id 0) (at 307.34 196.8205 0))
     (property "Value" "LT3469ETS8PBF" (id 1) (at 307.34 199.5956 0))
-    (property "Footprint" "Linear_Technology-LT3469ETS8PBF-*" (id 2) (at 297.815 191.135 0)
+    (property "Footprint" "Package_TO_SOT_SMD:TSOT-23-8" (id 2) (at 297.815 191.135 0)
       (effects (font (size 1.27 1.27)) (justify left) hide)
     )
@@
       (effects (font (size 1.27 1.27)) (justify left))
     )
-    (property "Footprint" "Fuse:Fuse_0603_1608Metric" (id 2) (at 241.3 68.58 90)
+    (property "Footprint" "libraries:C_FEEDTHRU_0603_TDK" (id 2) (at 241.3 68.58 90)
       (effects (font (size 1.27 1.27)) hide)
     )
@@
     (property "Reference" "Q1" (id 0) (at 154.94 34.7685 90))
     (property "Value" "Q_Dual_PMOS" (id 1) (at 154.94 37.5436 90))
-    (property "Footprint" "libraries:RESCAXE64P320X160X70-10N" (id 2) (at 154.94 41.91 0)
+    (property "Footprint" "" (id 2) (at 154.94 41.91 0)
       (effects (font (size 1.27 1.27)) hide)
     )
@@
     (property "Reference" "Q3" (id 0) (at 203.2 65.2485 90))
     (property "Value" "Q_Dual_PMOS" (id 1) (at 203.2 68.0236 90))
-    (property "Footprint" "libraries:RESCAXE64P320X160X70-10N" (id 2) (at 203.2 72.39 0)
+    (property "Footprint" "" (id 2) (at 203.2 72.39 0)
       (effects (font (size 1.27 1.27)) hide)
     )
@@
     (property "Reference" "Q2" (id 0) (at 180.34 52.5485 90))
     (property "Value" "Q_Dual_PMOS" (id 1) (at 180.34 55.3236 90))
-    (property "Footprint" "libraries:RESCAXE64P320X160X70-10N" (id 2) (at 180.34 59.69 0)
+    (property "Footprint" "" (id 2) (at 180.34 59.69 0)
       (effects (font (size 1.27 1.27)) hide)
     )
@@
     (property "Reference" "Q3" (id 0) (at 187.96 65.2485 90))
     (property "Value" "Q_Dual_PMOS" (id 1) (at 187.96 68.0236 90))
-    (property "Footprint" "libraries:RESCAXE64P320X160X70-10N" (id 2) (at 187.96 72.39 0)
-      (effects (font (size 1.27 1.27)) hide)
-    )
+    (property "Footprint" "" (id 2) (at 187.96 72.39 0)
+      (effects (font (size 1.27 1.27)) hide)
+    )
